File: stm32f103c8t6-circuit/f103c8t6开发板.kicad_pcb (KiCad board)
At the start: 2 copper layers, 40 x 40 mm, 46 parts, among them J1 Conn_01x04, J10 Conn_01x03, J11 Conn_01x03, J12 Conn_01x04, J13 Conn_01x04, J2 Conn_01x02, J3 Conn_01x03, J4 Conn_01x02, J5 USB_C_Receptacle_USB2.0, J6 Conn_01x06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

Commit message: Modify PCH and SCH
Parts:
- removed D5, D6: LED, LED_SMD:LED_0603_1608Metric
- removed J2: Conn_01x02, Connector_AMASS:AMASS_XT30UPB-M_1x02_P5.0mm_Vertical
- removed R10, R9: 1K, PCM_001_GN_RCL_SMD:R0603(1608M)
- removed R12, R13: 10k, PCM_001_GN_RCL_SMD:R0603(1608M)
- added D1: LED, LED_SMD:LED_0603_1608Metric, F.Cu at (160.4, 90.5)
- added D2: LED, LED_SMD:LED_0603_1608Metric, F.Cu at (160.4, 93.1)
- added R2: 1K, ResistorSMD:R_0603_1608Metric, F.Cu at (159.7, 83.5)
- added R3: 1K, ResistorSMD:R_0603_1608Metric, F.Cu at (163.7, 73.5)
- added R4: 10k, ResistorSMD:R_0603_1608Metric, F.Cu at (163.7, 76.0)
- added R5: 10k, ResistorSMD:R_0603_1608Metric, F.Cu at (163.7, 78.5)
- C1, C13, C14, C15, C16, C2, C3, C4, C5, C6: footprint PCM_001_GN_RCL_SMD:C0603(1608M) -> Capacitor_SMD:C_0603_1608Metric
- C20, C21: footprint Capacitor_SMD:C_0603_1608Metric_Pad1.08x0.95mm_HandSolder -> Capacitor_SMD:C_0603_1608Metric
- D4: value Diode_LED -> RED
- J1, J7: footprint PCM_205_CONN_GH_SMD:GH1.25_H_4 -> Connector_PinHeader_2.54mm:PinHeader_1x04_P2.54mm_Vertical
- R1, R11, R8: footprint PCM_001_GN_RCL_SMD:R0603(1608M) -> ResistorSMD:R_0603_1608Metric
- SW1, SW2, SW3: value (none) -> SW
- U1: footprint PCM_004_GN_MIDDLE-SEMI_SMD:QFP-48_7070 -> PackageQFP:LQFP-48_7x7mm_P0.5mm
- U3: footprint PCM_003_GN_SMALL-SEMI_SMD:SOT-23-5 -> PackageSOT:SOT-23-5
- Y1: footprint PCM_006_GN_XTAL_OSC_SMD:SMD-4_3225 -> Crystal:Crystal_SMD_3225-4Pin_3.2x2.5mm
- moved J1 34.0 mm to (110.4, 74.5)
- moved J6 31.9 mm to (114.6, 97.9)
- moved J10 23.9 mm to (119.7, 86.8)
- moved J9 23.9 mm to (115.1, 86.8)
- moved J11 23.9 mm to (124.4, 86.8)
- moved J3 23.9 mm to (110.4, 86.8)
- moved J4 23.8 mm to (130.7, 75.9)
- moved U5 23.8 mm to (130.4, 82.0)
- moved SW2 23.3 mm to (147.2, 79.8)
- moved SW3 23.3 mm to (147.2, 84.8)
- moved C17 20.8 mm to (136.7, 73.5)
- moved C19 20.8 mm to (136.7, 78.5)
- moved C18 20.8 mm to (136.7, 76.0)
- moved U1 20.6 mm to (146.4, 93.0)
- moved R8 19.6 mm to (142.7, 112.0)
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Connections:
- net /MCU/CAN_RX renamed /Connector/CAN_RX
- net /MCU/CAN_TX renamed /Connector/CAN_TX
- net /MCU/GPIO renamed /Connector/GPIO0
- net /MCU/PB1 renamed /MCU/KEY1
- net /MCU/PB12 renamed /Connector/PB12
- net /MCU/PB13 renamed /Connector/PB13
- net /MCU/PB14 renamed /Connector/PB14
- net /MCU/PB15 renamed /Connector/PB15
- net /MCU/PB2 renamed /MCU/KEY2
- net /MCU/RXD renamed /Connector/RXD
- net /MCU/SPI_CS renamed /Connector/SPI_CS
- net /MCU/SPI_MISO renamed /Connector/SPI_MISO
- net /MCU/SPI_MOSI renamed /Connector/SPI_MOSI
- net /MCU/SPI_SCK renamed /Connector/SPI_SCK
- net /MCU/TIM1_CH1 renamed /Connector/TIM1_CH
- net /MCU/TIM1_CH2 renamed /Connector/TIM1_CH2
- net /MCU/TIM2_CH1 renamed /Connector/TIM2_CH1
- net /MCU/TIM2_CH2 renamed /Connector/TIM2_CH2
- net /MCU/TXD renamed /Connector/TXD
- net /MCU/VCC renamed +3V3
- net /MCU/i2C1_SDA renamed /Connector/I2C1_SDA
- net /port/+ renamed /Connector/+
- net /port/- renamed /Connector/-
- net /port/DN renamed /Connector/DN
- net /port/DP renamed /Connector/DP
- C13 pad 2: /port/5V -> +5V
- C14 pad 2: /port/5V -> +5V
- C18 pad 2: /port/5V -> +5V
- C20 pad 1: /MCU/XTAL_I -> GND
- C20 pad 2: GND -> /MCU/XTAL_O
- C21 pad 1: /MCU/XTAL_O -> /MCU/XTAL_I
- J10 pad 1: /port/5V -> /Connector/5V
- J11 pad 1: /port/5V -> /Connector/5V
- J3 pad 1: /port/5V -> /Connector/5V
- J5 pad A4: /port/5V -> +5V
- J5 pad A9: /port/5V -> +5V
- J5 pad B4: /port/5V -> +5V
- J5 pad B9: /port/5V -> +5V
- J8 pad 3: /MCU/i2C1_SCL -> /Connector/I2C1_SCL
- J9 pad 1: /port/5V -> /Connector/5V
- U1 pad 42: /MCU/i2C1_SCL -> /MCU/I2C1_SCL
- U3 pad 1: /port/5V -> +5V
- U3 pad 3: /port/5V -> +5V
- U4 pad 3: /port/5V -> +5V

Commit message: Fix some SCH bugs
Connections:
- J10 pad 1: /Connector/5V -> +5V
- J11 pad 1: /Connector/5V -> +5V
- J3 pad 1: /Connector/5V -> +5V
- J9 pad 1: /Connector/5V -> +5V
- U1 pad 42: /MCU/I2C1_SCL -> /Connector/I2C1_SCL
