File: homework/rongjianchao/power.kicad_sch (KiCad schematic)
At the start: 7 parts, among them U3 HX9193-33GB

Commit message: 容键超2
Parts:
- U3: footprint PackageSOT:SOT-23-5 -> Package_TO_SOT_SMD:SOT-23-5_HandSoldering
Changed lines of the file:
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@@
       (effects (font (size 1.27 1.27)))
     )
-    (property "Footprint" "PackageSOT:SOT-23-5" (at 111.76 81.28 0)
+    (property "Footprint" "Package_TO_SOT_SMD:SOT-23-5_HandSoldering" (at 111.76 81.28 0)
       (effects (font (size 1.27 1.27)) hide)
     )
