File: homework/Lin Yuchuan/f103c8t6开发板.kicad_pcb (KiCad board)
At the start: 2 copper layers, 40 x 40 mm, 45 parts, among them J1 Conn_01x04, J10 Conn_01x03, J11 Conn_01x03, J12 Conn_01x04, J13 Conn_01x04, J3 Conn_01x03, J4 Conn_01x02, J5 USB_C_Receptacle_USB2.0, J6 Conn_01x06, J7 Conn_01x04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

Commit message: add silkscream
Parts:
- C17: moved to B.Cu
- moved C17 6.96 mm to (211.1, 84.5), turned to 180 degrees
- moved J5 2.23 mm to (185.7, 109.7)
- moved C18 2.15 mm to (193.7, 102.1)
- moved C1 1.26 mm to (185.7, 84.1)
- moved R1 0.96 mm to (185.7, 85.7)
- moved R5 0.41 mm to (213.4, 94.4)
- moved J12 0.15 mm to (206.2, 109.8)
- moved C14 0.09 mm to (186.6, 98.7)
- moved C13 0.07 mm to (184.8, 98.7)
Routing:
- net +3V3: track 195.5 -> 191.5 mm
- net /MCU/CLK: track 16.6 -> 20.3 mm
- net /Connector/DN: track 12.6 -> 16.2 mm
- net /Connector/DP: track 15.0 -> 16.6 mm
- net /MCU/DIO: track 19.3 -> 20.1 mm
- net /Connector/PB14: track 30.1 -> 30.7 mm
Other:
- board text added: "+3V3"
- board text added: "+5V"
- board text added: "3V3"
- board text added: "CLK"
- board text added: "DIO"
- board text added: "GND"
- board text added: "I2C1 SCL"
- board text added: "I2C1 SDA"
- board text added: "PB12"
- board text added: "PB13"
- board text added: "PB14"
- board text added: "PB15"
- board text added: "RXD"
- board text added: "TIM1 CH"
- board text added: "TIM1 CH2"
- board text added: "TIM2 CH1"
- board text added: "TIM2 CH2"
- board text added: "TXD"
